File: PowerMonitor.kicad_pcb (KiCad board)
At the start: 2 copper layers, 100 x 95 mm, 92 parts, among them J1 Conn_01x01, J10 TEST_1P, J11 TEST_1P, J12 TEST_1P, J13 TEST_1P, J14 TEST_1P, J15 TEST_1P, J16 Conn_01x03, J17 TEST_1P, J2 Conn_01x01, J3 Conn_01x01, J4 Conn_01x01, J5 Conn_01x01, J6 Conn_01x01, J7 Conn_01x01, J8 Conn_01x10, J9 TEST_1P, K1 T9AS5D12-5, K2 KEMET_UA2_5NJ, P1 Keystone_4912, P2 Keystone_4912, P3 Keystone_4912, P4 Keystone_4912, Q1 DMN3067LW, Q2 DMN3067LW, Q3 DMN3067LW, U1 IRM-02-5S, U2 IRM-05-5, U3 MCP39F521, U4 LP5907MFX-3.3, U5 ISO7731FDBQ, U6 ISO1540D

Commit message: Migrate to KiCAD nightly
Other:
- net class 0_4 removed
- net class 0_5 removed
- net class 3V_ISO removed
- net class 5V_ISO removed
- net class AC_L removed
- net class Default removed
- net class GND_ISO removed
